File: Platine/Zusatzplatine.brd (EAGLE design)
At the start: 77.1 x 52.1 mm, 25 parts

Commit message: - Platine weiter
Parts:
- removed D3: P6KEXXA, diode:C1702-15
- added D4: SM6T6V8A, diode:SMBG
- added DCF_3.3V, DCF_DATA, DCF_GND, DCF_POWON: SE14, solpad:SE14
- D1, D2: value 1N4148DO35-7 -> 1N4148WS; device diode:DO35-7 -> Diodes:SOD-323
- R1, R2: device rcl:0309/12 -> rcl:R1206
- moved D2 25.0 mm to (29.2, 38.1), flipped to the bottom, turned to 180 degrees
- moved D1 20.5 mm to (33.0, 38.1), flipped to the bottom, turned to 180 degrees
- moved R1 9.25 mm to (21.6, 27.9), flipped to the bottom, turned to 180 degrees
- moved WS_DIGOUT 6.48 mm to (30.5, 43.2)
- moved WLAN_3.3V 1.27 mm to (55.9, 38.1)
- flipped R2 to the bottom
Connections:
- removed net N$9: D2.A, D3.A
- new net N$17: DCF_GND.MP, JP2.9
- new net N$18: DCF_3.3V.MP, JP2.7
- new net N$19: DCF_POWON.MP, JP2.1
- new net N$20: DCF_DATA.MP, JP2.2
- net +3.3V: now also WLAN_3.3V.MP
- net N$10: now also D1.1, D4.C; no longer D1.C, D3.C
- net N$4: now also D2.0, D4.A
- net N$7: no longer D1.A, D2.C
- net N$8: now also D1.0, D2.1
Routing:
- net +3.3V: track 9.94 -> 59.8 mm
- net N$20: track 0.00 -> 24.4 mm
- net N$18: track 0.00 -> 23.0 mm
- net N$8: track 5.70 -> 24.3 mm
- net N$15: track 0.00 -> 15.5 mm
- net N$1: track 0.00 -> 13.5 mm
- net N$7: track 18.7 -> 31.8 mm
- net N$17: track 0.00 -> 13.0 mm
- net N$19: track 0.00 -> 12.0 mm
- net N$16: track 0.00 -> 11.7 mm
- net N$13: track 0.00 -> 11.4 mm
- net N$4: track 43.7 -> 54.0 mm
- net N$11: track 0.00 -> 9.20 mm
- net N$14: track 0.00 -> 7.62 mm
- net N$12: track 0.00 -> 7.62 mm
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Other:
- board size 77.1 x 52.1 mm -> 72.1 x 52.1 mm

Commit message: - kleine Änderungen - Beschriftungen
Parts:
- moved WLAN_3.3V 31.4 mm to (34.3, 61.0)
Routing:
- net +3.3V: track 59.8 -> 28.8 mm
- net N$4: track 54.0 -> 40.0 mm
- net N$5: track 64.9 -> 56.7 mm
Other:
- board text added: "DCF_33V"
- board text added: "DCF_DATA"
- board text added: "DCF_GND"
- board text added: "DCF_PD"
- board text added: "WLAN_33V"
- board text added: "WLAN_GND"
- board text added: "WLAN_GPIO0"
- board text added: "WLAN_GPIO1"
- board text added: "WLAN_PD"
- board text added: "WLAN_RST"
- board text added: "WLAN_RX"
- board text added: "WLAN_TX"
Changed lines of the file:
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@@
 <text x="25.541390625" y="58.98320625" size="0.8128" layer="16" rot="MR0">5V_IN</text>
 <text x="26.3430125" y="54.032271875" size="0.8128" layer="16" rot="MR0">5V_GND</text>
-<text x="26.085484375" y="40.74536875" size="0.8128" layer="16" rot="MR90">DIGOUT</text>
-<text x="26.13389375" y="33.590790625" size="0.8128" layer="16" rot="MR90">LED_GND</text>
-<text x="26.15926875" y="28.087828125" size="0.8128" layer="16" rot="MR90">LED_5V</text>
+<text x="27.355484375" y="42.01536875" size="0.8128" layer="16" rot="MR90">DIGOUT</text>
+<text x="24.86389375" y="38.670790625" size="0.8128" layer="16" rot="MR90">LED_GND</text>
+<text x="29.042209375" y="29.465940625" size="0.8128" layer="16" rot="MR0">LED_5V</text>
 <text x="22.14665" y="15.846790625" size="0.8128" layer="16" rot="MR180">LDR_IN</text>
 <text x="21.111325" y="20.87765625" size="0.8128" layer="16" rot="MR180">LDR_GND</text>
+<text x="45.72" y="59.69" size="0.8128" layer="16" rot="MR0">DCF_DATA</text>
+<text x="45.72" y="55.88" size="0.8128" layer="16" rot="MR0">DCF_33V</text>
+<text x="54.92926875" y="59.241265625" size="0.8128" layer="16" rot="MR0">DCF_PD</text>
+<text x="58.23878125" y="51.669396875" size="0.8128" layer="16" rot="MR0">DCF_GND</text>
+<text x="36.83" y="57.15" size="0.8128" layer="16" rot="MR0">WLAN_33V</text>
+<text x="58.42" y="34.29" size="0.8128" layer="16" rot="MR0">WLAN_GND</text>
+<text x="54.61" y="30.48" size="0.8128" layer="16" rot="MR0">WLAN_RST</text>
+<text x="58.42" y="26.67" size="0.8128" layer="16" rot="MR0">WLAN_GPIO1</text>
+<text x="54.61" y="24.13" size="0.8128" layer="16" rot="MR0">WLAN_GPIO0</text>
+<text x="58.42" y="20.32" size="0.8128" layer="16" rot="MR0">WLAN_PD</text>
+<text x="54.61" y="17.78" size="0.8128" layer="16" rot="MR0">WLAN_RX</text>
+<text x="58.42" y="13.97" size="0.8128" layer="16" rot="MR0">WLAN_TX</text>
 </plain>
 <attributes>
@@
 <element name="WS_DIGOUT" library="solpad" package="SE14" value="SE14" x="30.48" y="43.18"/>
 <element name="JP2" library="pinhead" package="2X19" value="" x="69.85" y="38.1" rot="R270"/>
-<element name="WLAN_3.3V" library="solpad" package="SE14" value="SE14" x="55.88" y="38.1"/>
+<element name="WLAN_3.3V" library="solpad" package="SE14" value="SE14" x="34.29" y="60.96"/>
 <element name="WLAN_GND" library="solpad" package="SE14" value="SE14" x="60.96" y="34.29"/>
 <element name="WLAN_TX" library="solpad" package="SE14" value="SE14" x="60.96" y="15.24"/>
@@
 <wire x1="16.6784" y1="53.1924" x2="16.51" y2="53.34" width="0.4" layer="16"/>
 <wire x1="23.964" y1="52.2876" x2="24.13" y2="52.07" width="0.4" layer="16"/>
-<wire x1="24.2656" y1="39.37" x2="17.45544375" y2="39.37" width="0.4064" layer="16"/>
-<wire x1="17.45544375" y1="39.37" x2="17.45544375" y2="44.723115625" width="0.4064" layer="16"/>
-<wire x1="17.45544375" y1="44.723115625" x2="24.182115625" y2="44.723115625" width="0.4064" layer="16"/>
 <wire x1="24.182115625" y1="44.723115625" x2="24.182115625" y2="44.8277125" width="0.4064" layer="16"/>
 <wire x1="24.182115625" y1="44.8277125" x2="24.13" y2="44.8277125" width="0.4064" layer="16"/>
@@
 <wire x1="27.31" y1="34.29" x2="24.13" y2="34.29" width="0.4064" layer="16"/>
 <wire x1="24.13" y1="34.29" x2="24.13" y2="36.83" width="0.4064" layer="16"/>
-<wire x1="27.31" y1="34.29" x2="28.11" y2="34.29" width="0.4064" layer="16"/>
-<wire x1="28.11" y1="34.29" x2="28.11" y2="38.1" width="0.4064" layer="16"/>
+<wire x1="27.31" y1="34.29" x2="28.11" y2="35.56" width="0.4064" layer="16"/>
+<wire x1="28.11" y1="35.56" x2="28.11" y2="38.1" width="0.4064" layer="16"/>
+<wire x1="24.182115625" y1="44.723115625" x2="24.2656" y2="44.723115625" width="0.4064" layer="16"/>
+<wire x1="24.2656" y1="44.723115625" x2="24.2656" y2="39.37" width="0.4064" layer="16"/>
 </signal>
 <signal name="N$5">
@@
 <wire x1="13.97" y1="52.07" x2="15.24" y2="50.8" width="0.4064" layer="16"/>
 <wire x1="15.24" y1="50.8" x2="19.05" y2="50.8" width="0.4064" layer="16"/>
-<wire x1="19.05" y1="50.8" x2="19.05" y2="45.72" width="0.4064" layer="16"/>
 <wire x1="21.59" y1="38.1" x2="21.59" y2="35.56" width="0.4064" layer="16"/>
 <wire x1="21.59" y1="35.56" x2="24.13" y2="33.02" width="0.4064" layer="16"/>
 <wire x1="24.13" y1="33.02" x2="24.13" y2="31.75" width="0.4064" layer="16"/>
-<wire x1="13.97" y1="38.252" x2="15.24" y2="43.18" width="0.4064" layer="16"/>
-<wire x1="15.24" y1="43.18" x2="15.24" y2="45.72" width="0.4064" layer="16"/>
-<wire x1="15.24" y1="45.72" x2="19.05" y2="45.72" width="0.4064" layer="16"/>
-<wire x1="21.59" y1="38.1" x2="15.24" y2="38.1" width="0.4064" layer="16"/>
-<wire x1="15.24" y1="38.1" x2="15.24" y2="43.18" width="0.4064" layer="16"/>
+<wire x1="21.59" y1="38.1" x2="19.05" y2="40.64" width="0.4064" layer="16"/>
+<wire x1="19.05" y1="40.64" x2="19.05" y2="50.8" width="0.4064" layer="16"/>
+<wire x1="13.97" y1="38.252" x2="16.358" y2="40.64" width="0.4064" layer="16"/>
+<wire x1="16.358" y1="40.64" x2="19.05" y2="40.64" width="0.4064" layer="16"/>
 </signal>
 <signal name="+3.3V">
@@
 <wire x1="16.51" y1="58.42" x2="20.32" y2="58.42" width="0.4064" layer="16"/>
 <wire x1="20.32" y1="58.42" x2="22.86" y2="60.96" width="0.4064" layer="16"/>
-<wire x1="22.86" y1="60.96" x2="33.02" y2="60.96" width="0.4064" layer="16"/>
-<wire x1="33.02" y1="60.96" x2="55.88" y2="38.1" width="0.4064" layer="16"/>
+<wire x1="22.86" y1="60.96" x2="34.29" y2="60.96" width="0.4064" layer="16"/>
 </signal>
 <signal name="N$6">

Commit message: - Platine Fehler behoben
Parts:
- moved R2 2.84 mm to (15.2, 34.3)
Connections:
- removed net N$5: 5V_IN.MP, JP1.6, R2.2, WS_5V.MP
- net N$10: now also 5V_IN.MP, JP1.6, R2.2, WS_5V.MP
Routing:
- net N$10: track 4.28 -> 84.2 mm
- net N$5: track 56.7 -> 0.00 mm
- net N$7: track 31.8 -> 22.7 mm
- net N$3: track 28.8 -> 26.6 mm
Changed lines of the file:
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@@
 <wire x1="75.87" y1="63.46579375" x2="3.81" y2="63.49" width="0" layer="20"/>
 <wire x1="3.81" y1="63.49" x2="3.81" y2="11.43" width="0" layer="20"/>
-<text x="15.189984375" y="54.171734375" size="0.8128" layer="16" rot="MR0">IR_GND</text>
-<text x="15.120278125" y="59.296996875" size="0.8128" layer="16" rot="MR0">IR_VDD</text>
-<text x="15.120278125" y="49.2556625" size="0.8128" layer="16" rot="MR0">IR_IN</text>
-<text x="25.541390625" y="58.98320625" size="0.8128" layer="16" rot="MR0">5V_IN</text>
-<text x="26.3430125" y="54.032271875" size="0.8128" layer="16" rot="MR0">5V_GND</text>
+<text x="22.696175" y="54.19208125" size="0.8128" layer="16" rot="MR0">IR_GND</text>
+<text x="16.390278125" y="60.566996875" size="0.8128" layer="16" rot="MR0">IR_VDD</text>
+<text x="13.87434375" y="49.76090625" size="0.8128" layer="16" rot="MR270">IR_IN</text>
+<text x="26.26354375" y="59.054415625" size="0.8128" layer="16" rot="MR0">5V_IN</text>
+<text x="29.8390875" y="49.111846875" size="0.8128" layer="16" rot="MR0">5V_GND</text>
 <text x="27.355484375" y="42.01536875" size="0.8128" layer="16" rot="MR90">DIGOUT</text>
-<text x="24.86389375" y="38.670790625" size="0.8128" layer="16" rot="MR90">LED_GND</text>
-<text x="29.042209375" y="29.465940625" size="0.8128" layer="16" rot="MR0">LED_5V</text>
+<text x="25.35211875" y="38.742" size="0.8128" layer="16" rot="MR90">LED_GND</text>
+<text x="29.3066625" y="29.150584375" size="0.8128" layer="16" rot="MR0">LED_5V</text>
 <text x="22.14665" y="15.846790625" size="0.8128" layer="16" rot="MR180">LDR_IN</text>
 <text x="21.111325" y="20.87765625" size="0.8128" layer="16" rot="MR180">LDR_GND</text>
@@
 <element name="LDR_GND" library="solpad" package="SE14" value="SE14" x="24.13" y="22.86"/>
 <element name="R1" library="rcl" package="R1206" value="120R" x="21.59" y="27.94" rot="MR180"/>
-<element name="R2" library="rcl" package="R1206" value="470R" x="13.97" y="36.83" rot="MR90"/>
+<element name="R2" library="rcl" package="R1206" value="470R" x="15.24" y="34.29" rot="MR90"/>
 <element name="WS_DIGOUT" library="solpad" package="SE14" value="SE14" x="30.48" y="43.18"/>
 <element name="JP2" library="pinhead" package="2X19" value="" x="69.85" y="38.1" rot="R270"/>
@@
 <wire x1="24.2656" y1="44.723115625" x2="24.2656" y2="39.37" width="0.4064" layer="16"/>
 </signal>
-<signal name="N$5">
-<contactref element="JP1" pad="6"/>
-<contactref element="5V_IN" pad="MP"/>
-<contactref element="WS_5V" pad="MP"/>
-<contactref element="R2" pad="2"/>
-<wire x1="22.7576" y1="55.9068" x2="10.3448" y2="55.9068" width="0.4" layer="16"/>
-<wire x1="23.964" y1="57.1132" x2="22.7576" y2="55.9068" width="0.4" layer="16"/>
-<wire x1="10.3448" y1="55.9068" x2="10.16" y2="55.88" width="0.4" layer="16"/>
-<wire x1="23.964" y1="57.1132" x2="24.13" y2="57.15" width="0.4" layer="16"/>
-<wire x1="23.964" y1="31.4772" x2="24.13" y2="31.75" width="0.4" layer="16"/>
-<wire x1="10.0432" y1="55.002" x2="10.0432" y2="55.6052" width="0.4" layer="16"/>
-<wire x1="8.8368" y1="53.7956" x2="10.0432" y2="55.002" width="0.4" layer="16"/>
-<wire x1="8.8368" y1="52.8908" x2="8.8368" y2="53.7956" width="0.4" layer="16"/>
-<wire x1="9.7416" y1="51.986" x2="8.8368" y2="52.8908" width="0.4" layer="16"/>
-<wire x1="10.0432" y1="55.6052" x2="10.16" y2="55.88" width="0.4" layer="16"/>
-<wire x1="9.7416" y1="51.986" x2="13.97" y2="51.986" width="0.4064" layer="16"/>
-<wire x1="13.97" y1="51.986" x2="13.97" y2="52.07" width="0.4064" layer="16"/>
-<wire x1="13.97" y1="52.07" x2="15.24" y2="50.8" width="0.4064" layer="16"/>
-<wire x1="15.24" y1="50.8" x2="19.05" y2="50.8" width="0.4064" layer="16"/>
-<wire x1="21.59" y1="38.1" x2="21.59" y2="35.56" width="0.4064" layer="16"/>
-<wire x1="21.59" y1="35.56" x2="24.13" y2="33.02" width="0.4064" layer="16"/>
-<wire x1="24.13" y1="33.02" x2="24.13" y2="31.75" width="0.4064" layer="16"/>
-<wire x1="21.59" y1="38.1" x2="19.05" y2="40.64" width="0.4064" layer="16"/>
-<wire x1="19.05" y1="40.64" x2="19.05" y2="50.8" width="0.4064" layer="16"/>
-<wire x1="13.97" y1="38.252" x2="16.358" y2="40.64" width="0.4064" layer="16"/>
-<wire x1="16.358" y1="40.64" x2="19.05" y2="40.64" width="0.4064" layer="16"/>
-</signal>
 <signal name="+3.3V">
 <contactref element="JP1" pad="5"/>
@@
 <wire x1="7.6304" y1="35.398" x2="7.62" y2="35.56" width="0.4" layer="16"/>
 <wire x1="23.964" y1="23.0324" x2="24.13" y2="22.86" width="0.4" layer="16"/>
-<wire x1="21.59" y1="34.1916" x2="21.59" y2="22.86" width="0.4064" layer="16"/>
 <wire x1="21.59" y1="22.86" x2="24.13" y2="22.86" width="0.4064" layer="16"/>
-<wire x1="9.7416" y1="34.1916" x2="21.59" y2="34.1916" width="0.4064" layer="16"/>
-<wire x1="21.59" y1="34.1916" x2="21.59" y2="34.29" width="0.4064" layer="16"/>
+<wire x1="9.7416" y1="34.1916" x2="9.84" y2="34.29" width="0.4064" layer="16"/>
+<wire x1="9.84" y1="34.29" x2="17.78" y2="34.29" width="0.4064" layer="16"/>
+<wire x1="17.78" y1="34.29" x2="21.59" y2="30.48" width="0.4064" layer="16"/>
+<wire x1="21.59" y1="30.48" x2="21.59" y2="22.86" width="0.4064" layer="16"/>
 </signal>
 <signal name="N$7">
 <contactref element="JP1" pad="34"/>
 <contactref element="R2" pad="1"/>
-<wire x1="18.7896" y1="28.0324" x2="14.2656" y2="28.0324" width="0.4" layer="16"/>
-<wire x1="14.2656" y1="28.0324" x2="13.97" y2="35.408" width="0.4" layer="16"/>
 <wire x1="10.0432" y1="21.2228" x2="10.0432" y2="20.6196" width="0.4" layer="16"/>
 <wire x1="8.8368" y1="22.4292" x2="10.0432" y2="21.2228" width="0.4" layer="16"/>
@@
 <wire x1="14.2656" y1="30.2708" x2="10.6464" y2="26.6516" width="0.4" layer="16"/>
 <wire x1="10.0432" y1="20.6196" x2="10.16" y2="20.32" width="0.4" layer="16"/>
-<wire x1="14.2656" y1="30.2708" x2="13.97" y2="35.408" width="0.4" layer="16"/>
 <contactref element="R1" pad="1"/>
 <wire x1="18.7896" y1="28.0324" x2="20.168" y2="28.0324" width="0.4064" layer="16"/>
 <wire x1="20.168" y1="28.0324" x2="20.168" y2="27.94" width="0.4064" layer="16"/>
+<wire x1="14.2656" y1="30.2708" x2="15.24" y2="31.2452" width="0.4064" layer="16"/>
+<wire x1="15.24" y1="31.2452" x2="15.24" y2="31.582" width="0.4064" layer="16"/>
+<wire x1="15.24" y1="31.75" x2="15.24" y2="32.868" width="0.4064" layer="16"/>
+<wire x1="18.7896" y1="28.0324" x2="15.24" y2="31.582" width="0.4064" layer="16"/>
+<wire x1="15.24" y1="31.582" x2="15.24" y2="31.75" width="0.4064" layer="16"/>
 </signal>
 <signal name="N$10">
@@
 <wire x1="33.65" y1="34.29" x2="34.12" y2="34.29" width="0.4064" layer="16"/>
 <wire x1="34.12" y1="34.29" x2="34.12" y2="38.1" width="0.4064" layer="16"/>
+<contactref element="WS_5V" pad="MP"/>
+<contactref element="5V_IN" pad="MP"/>
+<contactref element="JP1" pad="6"/>
+<contactref element="R2" pad="2"/>
+<wire x1="24.13" y1="57.15" x2="22.86" y2="55.88" width="0.4064" layer="16"/>
+<wire x1="22.86" y1="55.88" x2="10.16" y2="55.88" width="0.4064" layer="16"/>
+<wire x1="10.16" y1="55.88" x2="8.89" y2="54.61" width="0.4064" layer="16"/>
+<wire x1="8.89" y1="54.61" x2="8.89" y2="52.07" width="0.4064" layer="16"/>
+<wire x1="8.89" y1="52.07" x2="12.7" y2="52.07" width="0.4064" layer="16"/>
+<wire x1="12.7" y1="52.07" x2="13.97" y2="50.8" width="0.4064" layer="16"/>
+<wire x1="13.97" y1="50.8" x2="19.05" y2="50.8" width="0.4064" layer="16"/>
+<wire x1="19.05" y1="50.8" x2="19.05" y2="45.72" width="0.4064" layer="16"/>
+<wire x1="19.05" y1="45.72" x2="15.24" y2="41.91" width="0.4064" layer="16"/>
+<wire x1="15.24" y1="41.91" x2="15.24" y2="35.712" width="0.4064" layer="16"/>
+<wire x1="24.13" y1="57.15" x2="34.12" y2="47.16" width="0.4064" layer="16"/>
+<wire x1="34.12" y1="47.16" x2="34.12" y2="38.1" width="0.4064" layer="16"/>
+<wire x1="24.13" y1="31.75" x2="20.168" y2="35.712" width="0.4064" layer="16"/>
+<wire x1="20.168" y1="35.712" x2="15.24" y2="35.712" width="0.4064" layer="16"/>
 </signal>
 <signal name="N$1">

Commit message: - Platine überarbeitet
Parts:
- removed 5V_GND, 5V_IN: SE14, solpad:SE14
- added SUP_+5V, SUP_GND: SE14, solpad:SE14
- D4: device diode:SMBG -> diode:SMBJ
- moved LDR_GND 16.9 mm to (20.3, 39.4)
- moved LDR_IN 16.9 mm to (20.3, 34.3)
- moved R2 11.5 mm to (16.5, 22.9), turned to 270 degrees
- moved WS_5V 10.9 mm to (34.3, 27.9)
- moved WS_GND 8.98 mm to (25.4, 27.9)
- moved R1 3.81 mm to (21.6, 24.1)
- moved WLAN_3.3V 1.27 mm to (34.3, 59.7)
Connections:
- net N$7 renamed LED-OUT
- removed net N$10: 5V_IN.MP, D1.1, D4.C, JP1.6, R2.2, WS_5V.MP
- removed net N$16: JP2.20, WLAN_GND.MP
- removed net N$17: DCF_GND.MP, JP2.9
- new net +5V: D1.1, D4.C, JP1.6, R2.2, SUP_+5V.MP, WS_5V.MP
- new net GND: D2.0, D4.A, DCF_GND.MP, IR_GND.MP, JP1.20, JP1.22, JP1.8, JP2.20, JP2.9, SUP_GND.MP, WLAN_GND.MP, WS_GND.MP
- net N$4: now also JP1.19; no longer 5V_GND.MP, D2.0, D4.A, IR_GND.MP, JP1.8, WS_GND.MP
Routing:
- net N$10: track 84.2 -> 0.00 mm
- net +5V: track 0.00 -> 71.5 mm
- net N$4: track 40.0 -> 0.00 mm
- net N$17: track 13.0 -> 0.00 mm
- net N$3: track 26.6 -> 14.3 mm
- net N$16: track 11.7 -> 0.00 mm
- net LED-OUT: track 22.7 -> 18.9 mm
- net N$8: track 24.3 -> 28.1 mm
- net +3.3V: track 28.8 -> 28.0 mm
- added copper zone on layer 16, net GND
Other:
- board text added: "LED_OUT"
- board text added: "SUP_+5V"
- board text added: "SUP_GND"
- board text added: "WC-WS-Shield (c) 2015 K. Neumann"
- board text removed: "5V_GND"
- board text removed: "5V_IN"
- board text removed: "DIGOUT"
