File: Platine/Zusatzplatine.brd (EAGLE design)
At the start: 70 x 62.2 mm, 23 parts

Commit message: Platine: * WS-Schutz Layout verbessert * +5V & GND Leiterbahnen gelöscht (da wir Polygons haben) * DCF-In & DCF-PON auf Arduino Connector verlegt * kleine Trace-Umlegungen um Leitfähigkeit der Polygone zu verbessern * mehrere GND und einen +5V Pin mit entspr. Signalen verbunden
Dokumentation aktualisiert
Parts:
- moved D4 6.25 mm to (38.9, 53.6), turned to 0 degrees
- moved D1 4.57 mm to (40.6, 48.8), turned to 180 degrees
- moved D2 3.64 mm to (37.1, 48.8), turned to 180 degrees
Connections:
- removed net GND1: U$1.GND1
- removed net GND2: U$1.GND2
- removed net GND4: U$1.GND4
- removed net GND5: U$1.GND5
- removed net GND7: U$1.GND7
- removed net N$2: U$1.5V, U$1.5V2
- net +5V: now also U$1.5V, U$1.5V2
- net DCF1_DATA: now also U$1.D13; no longer U$1.PB9
- net DCF1_PON: now also U$1.D12; no longer U$1.PB8
- net GND: now also U$1.GND1, U$1.GND2, U$1.GND4, U$1.GND5, U$1.GND7
Routing:
- net GND: track 219.9 -> 9.40 mm, vias 4 -> 0
- net +5V: track 90.2 -> 30.0 mm, vias 1 -> 2
- net DCF1_PON: track 12.3 -> 24.2 mm
- net LED-OUT: track 71.0 -> 80.8 mm, vias 0 -> 3
- net DCF1_DATA: track 15.9 -> 20.6 mm
- net N$12: track 22.2 -> 25.8 mm
- net SWDIO: track 26.6 -> 29.1 mm
- net NRST: track 25.8 -> 28.1 mm
- net N$8: track 22.9 -> 24.2 mm, vias 0 -> 2
